File: Eagle_files/schematic2.brd (EAGLE design)
At the start: 101.6 x 53.3 mm, 77 parts, among them IC6 DS3231/SO

Commit message: I don't think I fixed much on this version, move to RevB for actual fixes.
Connections:
- net N$1 renamed XOUT+
- net N$19 renamed XOUT-
- net N$23 renamed YOUT-
- net N$24 renamed YOUT+
Changed lines of the file:
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@@
 <wire x1="50.8" y1="6.477" x2="51.943" y2="7.62" width="0.4064" layer="1"/>
 </signal>
-<signal name="N$19">
+<signal name="XOUT-">
 <contactref element="JOY_X" pad="2"/>
 <contactref element="JOYSTICK" pad="1"/>
@@
 <wire x1="55.118" y1="11.176" x2="55.118" y2="6.858" width="0.4064" layer="1"/>
 </signal>
-<signal name="N$23">
+<signal name="YOUT-">
 <contactref element="JOYSTICK" pad="3"/>
 <contactref element="JOY_Y" pad="2"/>
@@
 <wire x1="96.139" y1="21.59" x2="95.25" y2="21.59" width="0.4064" layer="1"/>
 </signal>
-<signal name="N$24">
+<signal name="YOUT+">
 <contactref element="JOYSTICK" pad="4"/>
 <contactref element="JOY_Y" pad="3"/>
@@
 <wire x1="23.038" y1="5.969" x2="22.971" y2="6.036" width="0.254" layer="1"/>
 </signal>
-<signal name="N$1">
+<signal name="XOUT+">
 <contactref element="JOYSTICK" pad="2"/>
 <contactref element="JOY_X" pad="3"/>
